File: PCB/OpenRemote.kicad_sch (KiCad schematic)
At the start: 172 parts, among them J1 USB_C_Receptacle_USB2.0, J2 Conn_01x50, J3 JST_PH_B2B-PH, J4 2.54x2 Header, J5 Micro_SD_Card, Q1 DMG2301L, Q2 MBT3904DW1, Q3 DMG2301L, Q4 DMG2301L, Q5 DMG2301L, Q6 FS8205A, Q7 DMG2301L, U1 DW01A, U10 APX803S, U11 TP4056, U12 TCA8418, U2 XC6220B331, U3 CH340C, U4 USBLC6-2P6, U5 LIS3DHTR, U6 TSSP77038, U7 ESP32-S3-WROOM-1-N16R8, U8 AP2112K-3.3, U9 MAX17048G

Commit message: Start Rev 6 Schematic
Parts:
- D2: footprint omoteLib:LED_5mm_Side_Mount -> OpenRemoteLib:LED_5mm_Side_Mount
- J1: footprint omoteLib:USB_C_Receptacle_HRO_TYPE-C-31-M-12 -> OpenRemoteLib:USB_C_Receptacle_HRO_TYPE-C-31-M-12
- J2: footprint omoteLib:TFT_2.83IN_240X320_50PIN -> OpenRemoteLib:TFT_2.83IN_240X320_50PIN; symbol omoteLib:Conn_01x50 -> OpenRemoteLib:Conn_01x50
- J3: footprint omoteLib:JST_PH_B2B-PH-SM4-TB_1x02-1MP_P2.00mm_Vertical -> OpenRemoteLib:JST_PH_B2B-PH-SM4-TB_1x02-1MP_P2.00mm_Vertical
- J5: footprint omoteLib:MicroSD Slot TF-01A -> OpenRemoteLib:MicroSD Slot TF-01A
- Q6: symbol omoteLib:FS8205A -> OpenRemoteLib:FS8205A
- U1: symbol omoteLib:DW01A -> OpenRemoteLib:DW01A
- U11: symbol omoteLib:TP4056 -> OpenRemoteLib:TP4056
- U12: symbol omoteLib:TCA8418 -> OpenRemoteLib:TCA8418
- U4: symbol omoteLib:USBLC6-2P6 -> OpenRemoteLib:USBLC6-2P6
- U5: symbol omoteLib:LIS3DHTR -> OpenRemoteLib:LIS3DHTR
- U6: footprint omoteLib:Heimdall vertical -> OpenRemoteLib:Heimdall vertical
- U9: symbol omoteLib:MAX17048G -> OpenRemoteLib:MAX17048G
Other:
- title: OMOTE - Open Universal Remote -> OpenRemote - Open Universal Remote

Commit message: Prepared to place mic on PCB
Parts:
- added MIC1: MS3625 Module, OpenRemoteLib:MS3625_Module_Back_Mount_SMD, symbol OpenRemoteLib:MS3625_Module
- added R45, R46, R47: 4k7, Resistor_SMD:R_0603_1608Metric, symbol Device:R
Connections:
- net GND: now also MIC1.1 (GND), MIC1.6 (L/R)
- net SD_MISO: now also R47.2
- net SD_MOSI: now also R46.2
- net SD_SCK: now also R45.2
- net MIC_VDD: now reaches D3.2 (A), U7.26 (IO45)
- net MIC_VDD: now also MIC1.2 (VDD)
- new net: MIC1.3 (SD), R47.1
- new net: MIC1.4 (SCK), R45.1
- new net: MIC1.5 (WS), R46.1
Other:
- note added: "I²S Microphone Module"
- note added: "RTC GPIO: 1–20; bootstraps: 0, 3, 45, 46 ext0: one RTC GPIO wake source ext1: multiple RTC GPIOs; any high or any low Internal pull-ups/pull-downs disabled"
- note removed: "RTC GPIO: 1-20 Bootstraps: 0,3,45,46 ext0: - single RTC_GPIO as wakeup source ext1: - multiple RTC_GPIOs as wakeup source - either any pin high or any pin low - internal Pull-ups /Pull-downs disabled"
- moved on the sheet: D3, R5
