File: PCB/Revision 6/OpenRemote.kicad_sch (KiCad schematic)
At the start: 176 parts, among them J1 USB_C_Receptacle_USB2.0, J2 Conn_01x50, J3 JST_PH_B2B-PH, J4 2.54x2 Header, J5 Micro_SD_Card, Q1 DMG2301L, Q2 MBT3904DW1, Q3 DMG2301L, Q4 DMG2301L, Q5 DMG2301L, Q6 FS8205A, Q7 DMG2301L, U1 DW01A, U10 APX803S, U11 TP4056, U12 TCA8418, U2 XC6220B331, U3 CH340C, U4 USBLC6-2P6, U5 LIS3DHTR, U6 TSSP77038, U7 ESP32-S3-WROOM-1-N16R8, U8 AP2112K-3.3, U9 MAX17048G

Commit message: Update Rev 6 project metadata
Other:
- company: Maximilian Kern -> Phillip Carlson
Changed lines of the file:
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@@
 	(title_block
 		(title "OpenRemote - Open Universal Remote")
-		(date "2024-12-22")
-		(rev "5")
-		(company "Maximilian Kern")
+		(date "5 Aug 2026")
+		(rev "6")
+		(company "Phillip Carlson")
 	)
 	(text "DB6"

Commit message: Add Rev 6 microphone and display updates
Parts:
- added J6: ER-CON06HB-1_TOUCH, OpenRemoteLib:ER-CON06HB-1_Compatible_1x06_P0.50mm_BottomContact, symbol OpenRemoteDisplay:ER-CON06HB-1_TOUCH
- added LCD1: Original Adafruit LCD assembly, OpenRemoteLib:Adafruit_280QV10_MECHANICAL, symbol Mechanical:MountingHole
- added LCD2: EastRising ER-TFT028-4.2 capacitive LCD, OpenRemoteLib:ER-TFT028-4.2_MECHANICAL, symbol Mechanical:MountingHole
Connections:
- net +VSW: now also J6.6 (+VSW)
- net GND: now also J6.1 (GND)
- net MIC_VDD: no longer D3.2 (A), U7.26 (IO45)
- net SCL: now also J6.3 (SCL)
- net SDA: now also J6.2 (SDA)
- net TP_NRST: now also J6.4 (TP_NRST)
- new net: D3.2 (A), U7.26 (IO45)
- no-connect marks 28 -> 29
