File: PCB/Revision 6/OpenRemote.kicad_sch (KiCad schematic)
At the start: 180 parts, among them J1 USB_C_Receptacle_USB2.0, J2 Conn_01x50, J3 JST_PH_B2B-PH, J4 2.54x2 Header, J5 Micro_SD_Card, J6 ER-CON06HB-1_TOUCH, J7 JST_PH_B2B-PH, Q1 DMG2301L, Q2 MBT3904DW1, Q3 DMG2301L, Q4 DMG2301L, Q5 DMG2301L, Q6 FS8205A, Q7 DMG2301L, U1 DW01A, U10 APX803S, U11 TP4056, U12 TCA8418, U2 XC6220B331, U3 CH340C, U4 USBLC6-2P6, U5 LIS3DHTR, U6 TSSP77038, U7 ESP32-S3-WROOM-1-N16R8, U8 AP2112K-3.3, U9 MAX17048G

Commit message: Add J6 assembly part code
Parts:
- J6: LCSC (none) -> C202118
Changed lines of the file:
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@@
+			)
+		)
+		(property "LCSC" "C202118"
+			(at 370.84 88.9 0)
+			(hide yes)
+			(show_name no)
+			(do_not_autoplace no)
+			(effects
+				(font
+					(size 1.27 1.27)
+				)
 			)
 		)
