File: PCB/Dock Rev6/Dock Rev6.kicad_sch (KiCad schematic)
At the start: 25 parts, among them J1 HX-XH2.54-2PZZ, Q1 FS8205A, SW1 KH-6X6X5H-ZJ, U1 ESP32-C3 Super Mini, U2 CC1101 433MHz COIL

Commit message: Restructure CAD around display variants, publish the Rev6 charging dock
CAD is now organised by what you print rather than by revision:

  CAD/Adafruit LCD/    3MF + STL set for the original Adafruit screen
  CAD/BuyDisplay LCD/  3MF + STL set for the EastRising/BuyDisplay screen
  CAD/Dock/            dock shell, base lid, menu button + 3MF
  CAD/*.f3z            current Fusion sources (remote v37/v38, dock v47)

The old CAD/Case Rev6 and CAD/Dock Rev6 trees are gone; their current
content is superseded by the v37/v47 exports. FusionScripts, Hardware
Models and PCB Imports keep their existing paths under CAD/.

Charging dock, published for the first time:
- Fusion source, printable parts and a Bambu 3MF
- KiCad project already present, now with a production set beside the
  gerbers: CPL.csv and a new BOM.xlsx
- README gains a Charging dock section covering pogo-pin charging, the
  ESP32-C3, the four-emitter IR bank, the CC1101 433 MHz radio and the
  power options

The dock BOM is generated from the board: 25 parts in 16 grouped lines,
matching the 25 CPL rows. LCSC codes come from the dock's own README
(C405273, C908265, C42391660, C2837541), from the PCB (C965807), and for
four passives from the remote BOM where value and footprint match exactly
(C1591, C15850, C22548, C98220). Ten designators still have no code -
100R, 100k, 100uF, the 39R IR resistors, and the two owner-supplied
modules - and are left blank rather than guessed.

Dock PCB sources also updated, plus the pre-FS8205A-fix board snapshots.

Note: CAD/Case Rev6/Community Parts (Case-Bulky-Bottom and the TPU
small-button variants) no longer exists on the source drive and is
removed here too. Restore with:
  git checkout 95b55f4 -- "CAD/Case Rev6/Community Parts"

Co-Authored-By: Claude Opus 5 <noreply@anthropic.com>
Connections:
- net IR_GATE: now also Q1.6 (G1); no longer Q1.2 (G1)
- net IR_K: now also Q1.2 (D1); no longer Q1.6 (D1)
Changed lines of the file:
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@@
+	(wire
+		(pts
+			(xy 22.86 55.88) (xy 27.94 55.88)
+		)
+		(stroke
+			(width 0)
+			(type default)
+		)
+	)
 	(wire
 		(pts
@@
 	(wire
 		(pts
+			(xy 35.56 55.88) (xy 38.1 55.88)
+		)
+		(stroke
+			(width 0)
+			(type default)
+		)
+	)
+	(wire
+		(pts
 			(xy 48.26 105.41) (xy 82.55 105.41)
 		)
@@
 	(wire
 		(pts
-			(xy 35.56 55.88) (xy 38.1 55.88)
-		)
-		(stroke
-			(width 0)
-			(type default)
-		)
-	)
-	(wire
-		(pts
 			(xy 91.44 26.67) (xy 107.95 26.67)
 		)
@@
 	(wire
 		(pts
-			(xy 27.94 41.91) (xy 55.88 41.91)
+			(xy 22.86 41.91) (xy 55.88 41.91)
 		)
 		(stroke
@@
 	(wire
 		(pts
-			(xy 27.94 41.91) (xy 27.94 55.88)
+			(xy 22.86 41.91) (xy 22.86 55.88)
 		)
 		(stroke

Commit message: Tidy the dock project and add D6 pogo-output protection diode
Cleanup - removed 21 files, keeping only the current board and
schematic. Everything remains in git history for rollback:
- 14 Dock Rev6.before-* rollback boards, schematics and prl
- Dock Rev6 Component Staging Backup.kicad_pcb
- 4 DRC/ERC/parity report files
- Dock Rev6.net and the exported Dock Rev6 Schematic.pdf

New diode, schematic only:
- D6, BAT20J Schottky, LCSC C49238173 - the same part as the remote's D1
- In series between +5V and J1 pin 1, creating the POGO_5V net, so the
  IR bank, ESP32 and decoupling stay on the raw 5V rail
- Orientation verified through the exported netlist: +5V carries D6 pin 2
  (A_2, anode) and POGO_5V carries D6 pin 1 (K_1, cathode) to J1 pin 1
- ERC passes with 0 violations

Deliberately NOT placed on the PCB - that is left to the owner.

Footprint and 3D model, project-local to match the dock's convention:
- project_libraries/footprints/DockRev6.pretty/D_SOD-323.kicad_mod
- project_libraries/3D-models/D_SOD-323.step
The footprint's model path is rewritten to ${KIPRJMOD}, so the project
does not depend on the global KiCad 3D model directory. The Diode symbol
library is added to sym-lib-table for the MBR0520 Schottky symbol, which
is what the remote uses for the same part.

The dock PCB also carries the owner's in-progress ESP32-C3 footprint
correction, untouched here.

Two caveats are recorded in the dock README: a series diode does not
limit current into a shorted pogo pair, and a BAT20J in SOD-323 is
marginal at the remote's ~1 A charge current.

Co-Authored-By: Claude Opus 5 <noreply@anthropic.com>
Parts:
- added D6: BAT20J, DockRev6:D_SOD-323, symbol Diode:MBR0520
Connections:
- net +5V: now also D6.2 (A); no longer J1.1
- new net POGO_5V: D6.1 (K), J1.1
Changed lines of the file:
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@@
 	(wire
 		(pts
-			(xy 88.9 52.07) (xy 88.9 63.5)
+			(xy 88.9 52.07) (xy 88.9 53.34)
+		)
+		(stroke
+			(width 0)
+			(type default)
+		)
+	)
+	(wire
+		(pts
+			(xy 88.9 60.96) (xy 88.9 63.5)
 		)
 		(stroke
@@
 					(unit 1)
 				)
+			)
+		)
+	)
+	(label "POGO_5V"
+		(at 88.9 62.23 0)
+		(fields_autoplaced yes)
+		(effects
+			(font
+				(size 1.27 1.27)
+			)
+			(justify left bottom)
+		)
+	)
+	(symbol
+		(lib_id "Diode:MBR0520")
+		(at 88.9 57.15 90)
+		(unit 1)
+		(exclude_from_sim no)
+		(in_bom yes)
+		(on_board yes)
+		(in_pos_files yes)
+		(dnp no)
+		(property "Reference" "D6"
+			(at 86.868 57.15 90)
+			(show_name no)
+			(do_not_autoplace no)
+			(effects
+				(font
+					(size 1.27 1.27)
+				)
+			)
+		)
+		(property "Value" "BAT20J"
+			(at 91.44 57.15 90)
+			(show_name no)
+			(do_not_autoplace no)
+			(effects
+				(font
+					(size 1.27 1.27)
+				)
+			)
+		)
+		(property "Footprint" "DockRev6:D_SOD-323"
+			(at 88.9 57.15 90)
+			(hide yes)
+			(show_name no)
+			(do_not_autoplace no)
+			(effects
+				(font
+					(size 1.27 1.27)
+				)
+			)
+		)
+		(property "Datasheet" "https://www.lcsc.com/datasheet/lcsc_datasheet_2410010330_STMicroelectronics-BAT20JFILM_C155590.pdf"
+			(at 88.9 57.15 0)
+			(hide yes)
+			(show_name no)
+			(do_not_autoplace no)
+			(effects
+				(font
+					(size 1.27 1.27)
+				)
+			)
+		)
+		(property "Description" "HIGH EFFICIENCY SWITCHING AND ULTRA LOW LEAKAGE CURRENT SCHOTTKY DIODE"
+			(at 88.9 57.15 0)
+			(hide yes)
+			(show_name no)
+			(do_not_autoplace no)
+			(effects
+				(font
+					(size 1.27 1.27)
+				)
+			)
+		)
+		(property "LCSC" "C49238173"
+			(at 88.9 57.15 0)
+			(hide yes)
+			(show_name no)
+			(do_not_autoplace no)
+			(effects
+				(font
+					(size 1.27 1.27)
+				)
+			)
+		)
+		(pin "1"
+		)
+		(pin "2"
+		)
+		(instances
+			(project "Dock Rev6"
+				(path "/67a795c7-71c1-4a83-b6d2-c7272e071e9d"
+					(reference "D6")
+					(unit 1)
+				)

Commit message: Replace the pogo diode with a 1A polyfuse
D6, the BAT20J Schottky added in the previous commit, is dropped in
favour of F1, a 1 A resettable polyfuse - the same part the remote uses
as its F1 (Device:Polyfuse, 1000mA, LCSC C220146).

It sits in the same place, in series between +5V and J1 pin 1 on the
POGO_5V net, with the IR bank, ESP32 and decoupling still on the raw 5V
rail. Still schematic only; not placed on the PCB.

Better suited to the job on both counts. A polyfuse trips on a shorted
pogo pair, which is the failure actually being guarded against and which
a series diode does nothing about. And it drops tens of millivolts
rather than roughly 0.45 V at 1 A, so the remote sees close to a full 5 V
instead of about 4.55 V.

The polyfuse symbol is vertical in the library with the same 7.62 mm pin
span as the diode, so it drops onto the existing wires unchanged, and
being non-polarised there is no orientation to get wrong.

Verified: ERC 0 violations, netlist shows +5V -> F1.1 and
POGO_5V -> F1.2 -> J1.1, and the sheet plots to PDF cleanly.

Also removes the now-unused diode footprint, its 3D model, the dead
Diode:MBR0520 lib_symbol left in the schematic, and the Diode entry in
sym-lib-table. The polyfuse footprint and 3D model are project-local like
the rest of the dock library.

README records the two remaining caveats: a polyfuse does not block
reverse current, and a 1 A hold part sits close to its limit at the
remote's ~1 A charge rate.

Co-Authored-By: Claude Opus 5 <noreply@anthropic.com>
Parts:
- removed D6: BAT20J, DockRev6:D_SOD-323, symbol Diode:MBR0520
- added F1: 1000mA, DockRev6:Fuse_1206_3216Metric_Pad1.42x1.75mm_HandSolder, symbol Device:Polyfuse
Connections:
- net +5V: now also F1.1
- net POGO_5V: now also F1.2
Changed lines of the file:
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@@
 	)
 	(symbol
-		(lib_id "Diode:MBR0520")
-		(at 88.9 57.15 90)
+		(lib_id "Device:Polyfuse")
+		(at 88.9 57.15 0)
 		(unit 1)
 		(exclude_from_sim no)
@@
 		(in_pos_files yes)
 		(dnp no)
-		(property "Reference" "D6"
-			(at 86.868 57.15 90)
+		(property "Reference" "F1"
+			(at 91.44 55.88 0)
 			(show_name no)
 			(do_not_autoplace no)
@@
 			)
 		)
-		(property "Value" "BAT20J"
-			(at 91.44 57.15 90)
+		(property "Value" "1000mA"
+			(at 91.44 58.42 0)
 			(show_name no)
 			(do_not_autoplace no)
@@
 			)
 		)
-		(property "Footprint" "DockRev6:D_SOD-323"
-			(at 88.9 57.15 90)
-			(hide yes)
-			(show_name no)
-			(do_not_autoplace no)
-			(effects
-				(font
-					(size 1.27 1.27)
-				)
-			)
-		)
-		(property "Datasheet" "https://www.lcsc.com/datasheet/lcsc_datasheet_2410010330_STMicroelectronics-BAT20JFILM_C155590.pdf"
+		(property "Footprint" "DockRev6:Fuse_1206_3216Metric_Pad1.42x1.75mm_HandSolder"
 			(at 88.9 57.15 0)
 			(hide yes)
@@
 			)
 		)
-		(property "Description" "HIGH EFFICIENCY SWITCHING AND ULTRA LOW LEAKAGE CURRENT SCHOTTKY DIODE"
+		(property "Datasheet" "~"
 			(at 88.9 57.15 0)
 			(hide yes)
@@
 			)
 		)
-		(property "LCSC" "C49238173"
+		(property "Description" "Resettable fuse, PPTC"
+			(at 88.9 57.15 0)
+			(hide yes)
+			(show_name no)
+			(do_not_autoplace no)
+			(effects
+				(font
+					(size 1.27 1.27)
+				)
+			)
+		)
+		(property "LCSC" "C220146"
 			(at 88.9 57.15 0)
 			(hide yes)
@@
 			(project "Dock Rev6"
 				(path "/67a795c7-71c1-4a83-b6d2-c7272e071e9d"
-					(reference "D6")
+					(reference "F1")
 					(unit 1)
 				)
